File: waveguide_simulation/kicad/waveguide.kicad_sch (KiCad schematic)
At the start: 2 parts

Commit message: experimented with meshing on planar waveguide
Parts:
- TP1: footprint TestPoint:TestPoint_Pad_1.0x1.0mm -> Resistor_SMD:R_0201_0603Metric
Changed lines of the file:
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@@
 			)
 		)
-		(property "Footprint" "TestPoint:TestPoint_Pad_1.0x1.0mm"
+		(property "Footprint" "Resistor_SMD:R_0201_0603Metric"
 			(at 46.99 101.6 0)
 			(effects
